File: Eagle Stuff/Mosaic/I2CConnector.brd (EAGLE design)
At the start: 45.4 x 7.6 mm, 2 parts

Commit message: DRC Adjustments
Parts:
- moved JP1 8.89 mm to (31.8, -1.27)
- moved JP2 8.89 mm to (31.8, 5.08)
Other:
- board size 45.4 x 7.6 mm -> 63.2 x 7.6 mm
Changed lines of the file:
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@@
 <setting verticaltext="up"/>
 </settings>
-<grid distance="50" unitdist="mil" unit="mil" style="lines" multiple="1" display="no" altdistance="5" altunitdist="mil" altunit="mil"/>
+<grid distance="50" unitdist="mil" unit="mm" style="lines" multiple="1" display="yes" altdistance="5" altunitdist="mil" altunit="mm"/>
 <layers>
 <layer number="1" name="Top" color="4" fill="1" visible="yes" active="yes"/>
@@
 <board>
 <plain>
-<wire x1="0" y1="0" x2="45.39" y2="0" width="0" layer="20"/>
-<wire x1="45.39" y1="0" x2="45.39" y2="7.61" width="0" layer="20"/>
-<wire x1="45.39" y1="7.61" x2="0" y2="7.61" width="0" layer="20"/>
+<wire x1="0" y1="0" x2="63.17" y2="0" width="0" layer="20"/>
+<wire x1="63.17" y1="0" x2="63.17" y2="7.61" width="0" layer="20"/>
+<wire x1="63.17" y1="7.61" x2="0" y2="7.61" width="0" layer="20"/>
 <wire x1="0" y1="7.61" x2="0" y2="0" width="0" layer="20"/>
 </plain>
@@
 </autorouter>
 <elements>
-<element name="JP2" library="pinhead" package="1X04" value="" x="22.86" y="5.08"/>
-<element name="JP1" library="pinhead" package="1X06/90" value="" x="22.86" y="-1.27" rot="R180"/>
+<element name="JP2" library="pinhead" package="1X04" value="" x="31.75" y="5.08"/>
+<element name="JP1" library="pinhead" package="1X06/90" value="" x="31.75" y="-1.27" rot="R180"/>
 </elements>
 <signals>
@@
 <contactref element="JP2" pad="4"/>
 <contactref element="JP1" pad="1"/>
-<wire x1="29.21" y1="2.54" x2="29.21" y2="5.08" width="0.8128" layer="16"/>
-<wire x1="29.21" y1="5.08" x2="26.67" y2="5.08" width="0.8128" layer="16"/>
+<wire x1="38.1" y1="2.54" x2="38.1" y2="5.08" width="0.8128" layer="16"/>
+<wire x1="38.1" y1="5.08" x2="35.56" y2="5.08" width="0.8128" layer="16"/>
 </signal>
 <signal name="VCC">
 <contactref element="JP2" pad="1"/>
 <contactref element="JP1" pad="6"/>
-<wire x1="16.51" y1="2.54" x2="16.51" y2="5.08" width="0.8128" layer="16"/>
-<wire x1="16.51" y1="5.08" x2="19.05" y2="5.08" width="0.8128" layer="16"/>
+<wire x1="25.4" y1="2.54" x2="25.4" y2="5.08" width="0.8128" layer="16"/>
+<wire x1="25.4" y1="5.08" x2="27.94" y2="5.08" width="0.8128" layer="16"/>
 </signal>
 <signal name="N$1">
 <contactref element="JP2" pad="3"/>
 <contactref element="JP1" pad="3"/>
-<wire x1="24.13" y1="2.54" x2="24.13" y2="5.08" width="0.8128" layer="16"/>
+<wire x1="33.02" y1="2.54" x2="33.02" y2="5.08" width="0.8128" layer="16"/>
 </signal>
 <signal name="N$2">
 <contactref element="JP2" pad="2"/>
 <contactref element="JP1" pad="4"/>
-<wire x1="21.59" y1="2.54" x2="21.59" y2="5.08" width="0.8128" layer="16"/>
+<wire x1="30.48" y1="2.54" x2="30.48" y2="5.08" width="0.8128" layer="16"/>
 </signal>
 </signals>
