File: Eagle Stuff/Mosaic/Master.brd (EAGLE design)
At the start: 54.6 x 63.2 mm, 9 parts

Commit message: DRC Adjustments
Other:
- board size 54.6 x 63.2 mm -> 53.3 x 63.2 mm
Changed lines of the file:
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@@
 <setting verticaltext="up"/>
 </settings>
-<grid distance="50" unitdist="mil" unit="mil" style="lines" multiple="1" display="no" altdistance="5" altunitdist="mil" altunit="mil"/>
+<grid distance="50" unitdist="mil" unit="mm" style="lines" multiple="1" display="yes" altdistance="5" altunitdist="mil" altunit="mm"/>
 <layers>
 <layer number="1" name="Top" color="4" fill="1" visible="yes" active="yes"/>
@@
 <board>
 <plain>
-<wire x1="0" y1="0" x2="54.59" y2="0" width="0" layer="20"/>
-<wire x1="54.59" y1="0" x2="54.59" y2="63.17" width="0" layer="20"/>
-<wire x1="54.59" y1="63.17" x2="0" y2="63.17" width="0" layer="20"/>
+<wire x1="0" y1="0" x2="53.32" y2="0" width="0" layer="20"/>
+<wire x1="53.32" y1="0" x2="53.32" y2="63.17" width="0" layer="20"/>
+<wire x1="53.32" y1="63.17" x2="0" y2="63.17" width="0" layer="20"/>
 <wire x1="0" y1="63.17" x2="0" y2="0" width="0" layer="20"/>
 </plain>
@@
 </signal>
 <signal name="N$5">
-<via x="48.26" y="57.15" extent="1-16" drill="3.048"/>
+<via x="48.26" y="58.42" extent="1-16" drill="3.048"/>
 </signal>
 <signal name="N$6">

Commit message: Final edits before etching
Routing:
- net GND: track 96.5 -> 102.0 mm
- net VCC: track 46.8 -> 48.3 mm
Changed lines of the file:
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@@
 <setting verticaltext="up"/>
 </settings>
-<grid distance="50" unitdist="mil" unit="mm" style="lines" multiple="1" display="yes" altdistance="5" altunitdist="mil" altunit="mm"/>
+<grid distance="50" unitdist="mil" unit="mil" style="lines" multiple="1" display="yes" altdistance="5" altunitdist="mil" altunit="mil"/>
 <layers>
 <layer number="1" name="Top" color="4" fill="1" visible="yes" active="yes"/>
@@
 <wire x1="35.56" y1="43.18" x2="38.1" y2="43.18" width="0.8128" layer="16"/>
 <wire x1="38.1" y1="43.18" x2="40.64" y2="43.18" width="0.8128" layer="16"/>
-<wire x1="14.3351875" y1="9.2456" x2="13.0556" y2="10.5251875" width="0.8128" layer="16"/>
-<wire x1="13.0556" y1="56.7848125" x2="14.3351875" y2="58.0644" width="0.8128" layer="16"/>
-<wire x1="15.24" y1="8.89" x2="14.8844" y2="9.2456" width="0.8128" layer="16"/>
-<wire x1="14.8844" y1="9.2456" x2="14.3351875" y2="9.2456" width="0.8128" layer="16"/>
+<wire x1="14.3351875" y1="58.0644" x2="13.0556" y2="56.7848125" width="0.8128" layer="16"/>
 <wire x1="14.3351875" y1="58.0644" x2="14.8844" y2="58.0644" width="0.8128" layer="16"/>
 <wire x1="14.8844" y1="58.0644" x2="15.24" y2="58.42" width="0.8128" layer="16"/>
-<wire x1="13.0556" y1="10.5251875" x2="13.0556" y2="56.7848125" width="0.8128" layer="16"/>
 <wire x1="15.24" y1="58.42" x2="15.24" y2="60.96" width="0.8128" layer="16"/>
 <wire x1="32.6644" y1="44.8056" x2="33.02" y2="44.45" width="0.8128" layer="16"/>
@@
 <wire x1="31.0292125" y1="60.96" x2="32.6644" y2="59.3248125" width="0.8128" layer="16"/>
 <wire x1="33.02" y1="44.45" x2="33.02" y2="43.18" width="0.8128" layer="16"/>
-<wire x1="13.0556" y1="10.5251875" x2="22.86" y2="25.4" width="0" layer="19" extent="16-16"/>
+<wire x1="13.97" y1="8.89" x2="13.0556" y2="9.8044" width="0.8128" layer="16"/>
+<wire x1="13.0556" y1="56.7848125" x2="13.0556" y2="9.8044" width="0.8128" layer="16"/>
+<wire x1="20.32" y1="8.89" x2="13.97" y2="8.89" width="0.8128" layer="16"/>
+<wire x1="20.32" y1="8.89" x2="22.86" y2="25.4" width="0" layer="19" extent="1-1"/>
 </signal>
 <signal name="N$1">
@@
 <wire x1="50.8" y1="35.56" x2="50.8" y2="38.1" width="0.8128" layer="16"/>
 <wire x1="50.8" y1="40.64" x2="50.8" y2="38.1" width="0.8128" layer="16"/>
-<wire x1="33.02" y1="35.56" x2="27.94" y2="35.56" width="0.8128" layer="16"/>
-<wire x1="27.94" y1="35.56" x2="27.94" y2="50.8" width="0.8128" layer="16"/>
-<wire x1="27.94" y1="50.8" x2="30.48" y2="53.34" width="0.8128" layer="16"/>
+<wire x1="27.94" y1="35.56" x2="33.02" y2="35.56" width="0.8128" layer="16"/>
+<wire x1="30.48" y1="53.34" x2="27.94" y2="53.34" width="0.8128" layer="16"/>
+<wire x1="27.94" y1="53.34" x2="27.94" y2="35.56" width="0.8128" layer="16"/>
 <wire x1="20.32" y1="25.4" x2="27.94" y2="35.56" width="0" layer="19" extent="16-16"/>
 </signal>
@@
 </signal>
 </signals>
+<errors>
+</errors>
 </board>
 </drawing>

Commit message: Fixed capacitor drill hole diameter
Parts:
- C1: value 10uF -> (none); device SparkFun-Capacitors:CPOL-RADIAL-2.5MM-5MM -> rcl:C025-030X050
- moved C1 1.27 mm to (27.9, 19.1), turned to 270 degrees
Routing:
- net N$4: track 40.7 -> 39.4 mm
- net N$3: track 3.83 -> 5.08 mm
Changed lines of the file:
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@@
 <element name="U$1" library="Teensy_3_and_LC_Series_Boards_v1.4" package="TEENSY_3.0-3.2&amp;LC_OUTER_ROW" value="TEENSY_3.1-3.2_OUTER_ROW" x="22.86" y="41.91"/>
 <element name="JP5" library="pinhead" package="1X05" value="" x="15.24" y="8.89" rot="R270"/>
-<element name="C1" library="SparkFun-Capacitors" package="CPOL-RADIAL-2.5MM-5MM" value="10uF" x="27.94" y="20.32" rot="R90">
-<attribute name="PROD_ID" value="CAP-08440" x="27.94" y="20.32" size="1.778" layer="27" rot="R90" display="off"/>
-</element>
+<element name="C1" library="rcl" package="C025-030X050" value="" x="27.94" y="19.05" rot="R270"/>
 </elements>
 <signals>
@@
 <contactref element="U$1" pad="RESET/DAC"/>
 <contactref element="C1" pad="1"/>
-<wire x1="27.94" y1="21.57" x2="27.94" y2="25.4" width="0.8128" layer="16"/>
+<wire x1="27.94" y1="20.32" x2="27.94" y2="25.4" width="0.8128" layer="16"/>
 </signal>
 <signal name="N$4">
-<contactref element="C1" pad="2"/>
 <contactref element="JP5" pad="1"/>
 <contactref element="JP5" pad="5"/>
-<wire x1="27.94" y1="13.97" x2="27.94" y2="19.07" width="0.8128" layer="16"/>
 <wire x1="27.94" y1="13.97" x2="15.24" y2="13.97" width="0.8128" layer="16"/>
 <wire x1="15.24" y1="3.81" x2="27.94" y2="3.81" width="0.8128" layer="16"/>
 <wire x1="27.94" y1="3.81" x2="27.94" y2="13.97" width="0.8128" layer="16"/>
+<contactref element="C1" pad="2"/>
+<wire x1="27.94" y1="17.78" x2="27.94" y2="13.97" width="0.8128" layer="16"/>
 </signal>
 <signal name="N$5">
